File: hw/sch_pcb/RETERMINT01.kicad_pcb (KiCad board)
At the start: 2 copper layers, 89.6 x 119.5 mm, 83 parts, among them J1 Conn_02x05_Odd_Even, J10 Raspberry_Pi_4, J11 RJ45_LED_Shielded, J2 Barrel_Jack_Switch, J3 HEADER_2x05_PARALLEL, J4 HEADER_2x01_PARALLEL, J5 HEADER_2x01_PARALLEL, J6 HEADER_2x01_PARALLEL, J7 HEADER_2x01_PARALLEL, J8 u.fl, J9 HEADER_2x01_PARALLEL, M1 HOLE, M2 HOLE, M3 HOLE, M4 HOLE, Q1 BC817-25, Q2 BC817-25, U1 TPSM33606S5QRDNRQ1, U2 USBLC6-2SC6, U3 MIC5504-3.3YM5, U4 NEO-M9N, U5 ADM2483xRW, U6 ADM2483xRW, U7 ADM2483xRW

Commit message: Update component values.
Parts:
- C11, C2, C4: value 1u -> 1uF
- C12, C3: value 100n -> 100nF
Changed lines of the file:
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@@
 			)
 		)
-		(property "UST_ID" ""
+		(property "UST_ID" "5c70984512875079b91f898c"
 			(at 0 0 0)
 			(unlocked yes)
@@
 			)
 		)
-		(property "Value" "100n"
+		(property "Value" "100nF"
 			(at 0 1.679999 0)
 			(layer "F.Fab")
@@
 			)
 		)
+		(property "UST_ID" "5c70984712875079b91f8b4c"
+			(at 0 0 180)
+			(unlocked yes)
+			(layer "F.Fab")
+			(hide yes)
+			(effects
+				(font
+					(size 1 1)
+					(thickness 0.15)
+				)
+			)
+		)
 		(property ki_fp_filters "C_*")
 		(sheetname "/")
@@
 			)
 		)
-		(property "UST_ID" ""
+		(property "UST_ID" "5c70984612875079b91f899f"
 			(at 0 0 180)
 			(unlocked yes)
@@
 			)
 		)
-		(property "Value" "1u"
+		(property "Value" "1uF"
 			(at 0 1.68 0)
 			(layer "F.Fab")
@@
 			)
 		)
+		(property "UST_ID" "5c70984712875079b91f8b50"
+			(at 0 0 0)
+			(unlocked yes)
+			(layer "F.Fab")
+			(hide yes)
+			(effects
+				(font
+					(size 1 1)
+					(thickness 0.15)
+				)
+			)
+		)
 		(property ki_fp_filters "C_*")
 		(sheetname "/")
@@
 			)
 		)
-		(property "UST_ID" ""
+		(property "UST_ID" "5c70984612875079b91f899f"
 			(at 0 0 0)
 			(unlocked yes)
@@
 			)
 		)
-		(property "Value" "1u"
+		(property "Value" "1uF"
 			(at 0 1.679999 90)
 			(layer "F.Fab")
@@
 			)
 		)
+		(property "UST_ID" "5c70984712875079b91f8b50"
+			(at 0 0 270)
+			(unlocked yes)
+			(layer "F.Fab")
+			(hide yes)
+			(effects
+				(font
+					(size 1 1)
+					(thickness 0.15)
+				)
+			)
+		)
 		(property ki_fp_filters "C_*")
 		(sheetname "/")
@@
 			)
 		)
-		(property "Value" "100n"
+		(property "Value" "100nF"
 			(at 0 1.679999 0)
 			(layer "F.Fab")
@@
 			)
 		)
+		(property "UST_ID" "5c70984712875079b91f8b4c"
+			(at 0 0 180)
+			(unlocked yes)
+			(layer "F.Fab")
+			(hide yes)
+			(effects
+				(font
+					(size 1 1)
+					(thickness 0.15)
+				)
+			)
+		)
 		(property ki_fp_filters "C_*")
 		(sheetname "/")
@@
 			)
 		)
+		(property "UST_ID" "?"
+			(at 0 0 90)
+			(unlocked yes)
+			(layer "F.Fab")
+			(hide yes)
+			(effects
+				(font
+					(size 1 1)
+					(thickness 0.15)
+				)
+			)
+		)
 		(property ki_fp_filters "SOT?23*")
 		(sheetname "/")
@@
 			)
 		)
-		(property "Value" "1u"
+		(property "Value" "1uF"
 			(at 0 1.679999 0)
 			(layer "F.Fab")
@@
 			)
 		)
+		(property "UST_ID" "5c70984712875079b91f8b50"
+			(at 0 0 180)
+			(unlocked yes)
+			(layer "F.Fab")
+			(hide yes)
+			(effects
+				(font
+					(size 1 1)
+					(thickness 0.15)
+				)
+			)
+		)
 		(property ki_fp_filters "C_*")
 		(sheetname "/")
@@
 			)
 		)
-		(property "UST_ID" ""
+		(property "UST_ID" "5fa0faaf12875025b3977985"
 			(at 0 0 270)
 			(unlocked yes)
@@
 			)
 		)
+		(property "UST_ID" "5ed7ac8e12875004e15a62c8"
+			(at 0 0 0)
+			(unlocked yes)
+			(layer "F.Fab")
+			(hide yes)
+			(effects
+				(font
+					(size 1 1)
+					(thickness 0.15)
+				)
+			)
+		)
 		(property ki_fp_filters "*BNC* *SMA* *SMB* *SMC* *Cinch* *LEMO* *UMRF* *MCX* *U.FL*")
 		(sheetname "/")
@@
 	)
 	(segment
+		(start 69 96.8)
+		(end 69 82.31)
+		(width 0.3)
+		(layer "F.Cu")
+		(net "/PWR_ON")
+	)
+	(segment
+		(start 78.4 106.2)
+		(end 69 96.8)
+		(width 0.3)
+		(layer "F.Cu")
+		(net "/PWR_ON")
+	)
+	(segment
+		(start 82.175 120.3)
+		(end 81.2 120.3)
+		(width 0.3)
+		(layer "F.Cu")
+		(net "/PWR_ON")
+	)
+	(segment
+		(start 69 82.31)
+		(end 67.725 81.035)
+		(width 0.3)
+		(layer "F.Cu")
+		(net "/PWR_ON")
+	)
+	(segment
+		(start 78.4 117.5)
+		(end 78.4 106.2)
+		(width 0.3)
+		(layer "F.Cu")
+		(net "/PWR_ON")
+	)
+	(segment
+		(start 81.2 120.3)
+		(end 78.4 117.5)
+		(width 0.3)
+		(layer "F.Cu")
+		(net "/PWR_ON")
+	)
+	(segment
 		(start 84 118.2125)
 		(end 84.0125 118.2)
@@
 		(net "Net-(Q2-B)")
 	)
-	(segment
-		(start 69 96.8)
-		(end 69 82.31)
-		(width 0.3)
-		(layer "F.Cu")
-		(net "/PWR_ON")
-	)
-	(segment
-		(start 78.4 106.2)
-		(end 69 96.8)
-		(width 0.3)
-		(layer "F.Cu")
-		(net "/PWR_ON")
-	)
-	(segment
-		(start 82.175 120.3)
-		(end 81.2 120.3)
-		(width 0.3)
-		(layer "F.Cu")
-		(net "/PWR_ON")
-	)
-	(segment
-		(start 69 82.31)
-		(end 67.725 81.035)
-		(width 0.3)
-		(layer "F.Cu")
-		(net "/PWR_ON")
-	)
-	(segment
-		(start 78.4 117.5)
-		(end 78.4 106.2)
-		(width 0.3)
-		(layer "F.Cu")
-		(net "/PWR_ON")
-	)
-	(segment
-		(start 81.2 120.3)
-		(end 78.4 117.5)
-		(width 0.3)
-		(layer "F.Cu")
-		(net "/PWR_ON")
-	)
 	(zone

Commit message: fix issues
Parts:
- added C13: 100nF, Capacitor_SMD:C_0805_2012Metric, F.Cu at (136.4, 115.3)
- added C14: 100nF, Capacitor_SMD:C_0805_2012Metric, F.Cu at (103.3, 127.5)
- added C15: 100nF, Capacitor_SMD:C_0805_2012Metric, F.Cu at (125.7, 115.4)
- added C16: 100nF, Capacitor_SMD:C_0805_2012Metric, F.Cu at (125.8, 131.6)
- added C17: 100nF, Capacitor_SMD:C_0805_2012Metric, F.Cu at (114.8, 115.4)
- added C18: 100nF, Capacitor_SMD:C_0805_2012Metric, F.Cu at (136.1, 132.6)
- moved J1 14.5 mm to (125.1, 42.6), turned to -90 degrees
- moved U2 3.80 mm to (121.5, 49.0), turned to 90 degrees
- moved J10 0.56 mm to (67.7, 46.0)
Connections:
- J10 pad 18: unconnected-(J10-GPIO24/SDIO_DAT0-Pad18) -> /TIMEPULSE
- J10 pad 22: unconnected-(J10-GPIO25/SDIO_DAT1-Pad22) -> /PWR_ON
- J10 pad 29: /PWR_ON -> unconnected-(J10-GPCLK1/GPIO05-Pad29)
- J10 pad 7: /TIMEPULSE -> unconnected-(J10-GPCLK0/GPIO04-Pad7)
- JP3 pad 2: /ch3_vdd -> Net-(JP3-C)
- JP3 pad 3: +3V3_DIG -> +3V3
- U5 pad 1: +3V3_DIG -> +3V3
- U5 pad 4: +3V3_DIG -> +3V3
- U5 pad 5: +3V3_DIG -> +3V3
- U6 pad 1: +3V3_DIG -> +3V3
- U7 pad 1: /ch3_vdd -> +3V3
- U7 pad 4: /ch3_vdd -> Net-(JP3-C)
- U7 pad 5: /ch3_vdd -> Net-(JP3-C)
Routing:
- net +3V3: track 148.8 -> 246.9 mm, vias 6 -> 10
- net +3V3_DIG: track 53.6 -> 0.00 mm, vias 2 -> 0
- net /ch3_vdd: track 17.8 -> 0.00 mm
- net GND_DIG: track 17.8 -> 30.0 mm, vias 28 -> 33
- net /VBUS: track 16.7 -> 28.0 mm
- net /PWR_ON: track 45.8 -> 55.4 mm
- net Net-(JP3-C): track 0.00 -> 8.88 mm
- net +5V_OUT: track 64.4 -> 68.1 mm
- net /TIMEPULSE: track 80.4 -> 82.2 mm, vias 3 -> 2
- net /D1P: track 4.91 -> 3.23 mm
- net /D1M: track 3.14 -> 4.80 mm
- net GND_GPS: track 18.1 -> 17.0 mm, vias 24 -> 23
- net /D1-: track 3.57 -> 2.75 mm
- net /TX: track 87.1 -> 86.3 mm
- net unconnected-(J10-GPCLK1/GPIO05-Pad29): track 0.00 -> 0.56 mm
Other:
- board text added: "2026/06 roman-dvorak"
- board text added: "PWR"
- board text added: "RETERMINT01B"
- board text added: "RX"
- board text added: "TPS"
- board text added: "TX"
- board text removed: "2026"
- board text removed: "RETERMINT01A"
